Commit message: feat: Newthon Raphson first implementation

File: src/catkin_ws/src/Jackal-UWB-custom/urdf/jackal_custom/custom_jackal.urdf.xacro (robot description, xacro)
@@ -4,6 +4,8 @@
     <xacro:arg name="right_id" default="0" />
     <xacro:arg name="left_id" default="1" />
+    <xacro:arg name="rear_id" default="2" />
     <xacro:property name="right" value="$(arg right_id)" />
     <xacro:property name="left" value="$(arg left_id)" />
+    <xacro:property name="rear" value="$(arg rear_id)" />
     <link name="right_tag">
         <inertial>
@@ -68,4 +70,34 @@
         <material>Gazebo/White</material>
     </gazebo>
+    <link name="rear_tag">
+        <inertial>
+            <mass value="0.1" />
+            <origin rpy="0 0 0" xyz="0 0 0"/>
+            <inertia ixx="1.0" ixy="0.0" ixz="0.0" iyy="1.0" iyz="0.0" izz="1.0" />
+        </inertial>
+        <collision>
+            <origin xyz="0 -0.013 0" rpy="0 0 0"/>
+            <geometry>
+                <box size="0.05 0.026 0.102"/>
+            </geometry>
+        </collision>
+        <visual>
+            <origin xyz="0 0 0" rpy="0 0 0"/>
+            <geometry>
+                <mesh filename="package://jackal-custom/models/DecaWave/meshes/Decawave.stl"/>
+            </geometry>
+        </visual>
+    </link>
+    <joint name="rear_tag_joint" type="fixed">
+        <origin xyz="-0.2155 0 0.184" rpy="-0.78 0 -1.57"/>
+        <parent link="base_link"/>
+        <child link="rear_tag"/>
+    </joint>
+    <gazebo reference="rear_tag_joint">
+        <preserveFixedJoint>true</preserveFixedJoint>
+    </gazebo>
+    <gazebo reference="rear_tag">
+        <material>Gazebo/White</material>
+    </gazebo>
     <gazebo>
         <plugin name='libgtec_uwb_plugin' filename='libgtec_uwb_plugin.so'>
@@ -77,8 +109,9 @@
             <anchor_prefix>uwb_anchor</anchor_prefix>
             <tag_id>${right}</tag_id>
-            <noise type='gaussian'>
+            <!-- Not sure this is necessary. The UWB noise model is already in UWBPlugin.cpp-->
+            <!--noise type='gaussian'>
                 <mean>0</mean>
                 <stddev>0.0</stddev>
-            </noise>
+            </noise-->
         </plugin>
     </gazebo>
@@ -92,8 +125,25 @@
             <anchor_prefix>uwb_anchor</anchor_prefix>
             <tag_id>${left}</tag_id>
-            <noise type='gaussian'>
+            <!-- Not sure this is necessary. The UWB noise model is already in UWBPlugin.cpp-->
+            <!--noise type='gaussian'>
                 <mean>0</mean>
                 <stddev>0.0</stddev>
-            </noise>
+            </noise-->
+        </plugin>
+    </gazebo>
+    <gazebo>
+        <plugin name='libgtec_uwb_plugin' filename='libgtec_uwb_plugin.so'>
+            <update_rate>5</update_rate>
+            <frequency>3.9936e9</frequency>
+            <power>-14.3</power>
+            <rx_gain>2</rx_gain>
+            <tag_link>rear_tag</tag_link>
+            <anchor_prefix>uwb_anchor</anchor_prefix>
+            <tag_id>${rear}</tag_id>
+            <!-- Not sure this is necessary. The UWB noise model is already in UWBPlugin.cpp-->
+            <!--noise type='gaussian'>
+                <mean>0</mean>
+                <stddev>0.0</stddev>
+            </noise-->
         </plugin>
     </gazebo>

Commit message: feat: remove uwb-plugin dependence

File: src/catkin_ws/src/Jackal-UWB-custom/urdf/jackal_custom/custom_jackal.urdf.xacro (robot description, xacro)
@@ -2,10 +2,11 @@
 <robot xmlns:xacro="http://www.ros.org/wiki/xacro" name="Jackal">
     <xacro:include filename="$(find jackal-custom)/urdf/jackal_custom/custom_jackal_base.urdf.xacro" />
-    <xacro:arg name="right_id" default="0" />
-    <xacro:arg name="left_id" default="1" />
-    <xacro:arg name="rear_id" default="2" />
-    <xacro:property name="right" value="$(arg right_id)" />
-    <xacro:property name="left" value="$(arg left_id)" />
+    <xacro:arg name="rear_id" default="0" />
+    <!--xacro:arg name="right_id" default="1" /-->
+    <!--xacro:arg name="left_id" default="2" /-->
+    <!--xacro:property name="right" value="$(arg right_id)" /-->
+    <!--xacro:property name="left" value="$(arg left_id)" /-->
     <xacro:property name="rear" value="$(arg rear_id)" />
+    <!--
     <link name="right_tag">
         <inertial>
@@ -29,5 +30,4 @@
     <joint name="right_tag_joint" type="fixed">
         <origin xyz="0 -0.161786 0.184" rpy="0 0 0"/>
-        <!-- <origin xyz="0 0.161786 0" rpy="0 0 3.14159265359"/> -->
         <parent link="base_link"/>
         <child link="right_tag"/>
@@ -39,4 +39,6 @@
         <material>Gazebo/White</material>
     </gazebo>
+    -->
+    <!--
     <link name="left_tag">
         <inertial>
@@ -60,5 +62,4 @@
     <joint name="left_tag_joint" type="fixed">
         <origin xyz="0 0.161786 0.184" rpy="0 0 3.14159265359"/>
-        <!-- <origin xyz="0 -0.161786 0" rpy="0 0 0"/> -->
         <parent link="base_link"/>
         <child link="left_tag"/>
@@ -70,4 +71,5 @@
         <material>Gazebo/White</material>
     </gazebo>
+    -->
     <link name="rear_tag">
         <inertial>
@@ -90,6 +92,7 @@
     </link>
     <joint name="rear_tag_joint" type="fixed">
-        <origin xyz="-0.2155 0 0.184" rpy="-0.78 0 -1.57"/>
-        <!--origin xyz="-0.5 0 0.184" rpy="0 0 -1.57"/-->
+        <!--origin xyz="-0.2155 0 0.184" rpy="-0.78 0 -1.57"/-->
+        <!--origin xyz="-0.5 0 0.184" rpy="0 0 0"/-->
+        <origin xyz="-0.5 0 0.184" rpy="0 0 -1.57"/>
         <parent link="base_link"/>
         <child link="rear_tag"/>
@@ -101,4 +104,5 @@
         <material>Gazebo/White</material>
     </gazebo>
+    <!--
     <gazebo>
         <plugin name='libgtec_uwb_plugin' filename='libgtec_uwb_plugin.so'>
@@ -110,11 +114,8 @@
             <anchor_prefix>uwb_anchor</anchor_prefix>
             <tag_id>${right}</tag_id>
-            <!-- Not sure this is necessary. The UWB noise model is already in UWBPlugin.cpp-->
-            <!--noise type='gaussian'>
-                <mean>0</mean>
-                <stddev>0.0</stddev>
-            </noise-->
         </plugin>
     </gazebo>
+    -->
+    <!--
     <gazebo>
         <plugin name='libgtec_uwb_plugin' filename='libgtec_uwb_plugin.so'>
@@ -126,11 +127,8 @@
             <anchor_prefix>uwb_anchor</anchor_prefix>
             <tag_id>${left}</tag_id>
-            <!-- Not sure this is necessary. The UWB noise model is already in UWBPlugin.cpp-->
-            <!--noise type='gaussian'>
-                <mean>0</mean>
-                <stddev>0.0</stddev>
-            </noise-->
         </plugin>
     </gazebo>
+    -->
+    <!--
     <gazebo>
         <plugin name='libgtec_uwb_plugin' filename='libgtec_uwb_plugin.so'>
@@ -142,11 +140,7 @@
             <anchor_prefix>uwb_anchor</anchor_prefix>
             <tag_id>${rear}</tag_id>
-            <!-- Not sure this is necessary. The UWB noise model is already in UWBPlugin.cpp-->
-            <!--noise type='gaussian'>
-                <mean>0</mean>
-                <stddev>0.0</stddev>
-            </noise-->
         </plugin>
     </gazebo>
+    -->
     <gazebo>
         <plugin name="p3d_base_controller" filename="libgazebo_ros_p3d.so">
