Commit message: feat: only one EKF, no user tf publishing

File: src/catkin_ws/src/jackal-custom/urdf/custom_jackal_base.urdf.xacro (robot description, xacro)
@@ -74,4 +74,10 @@
     <child link="world" />
   </joint>
+  <link name="odom"></link>
+  <joint name="odom_joint" type="fixed">
+    <origin xyz="0 0 0" rpy="0 0 0" />
+    <parent link="odom"/>
+    <child link="base_link" />
+  </joint>
   <link name="base_link"></link>
   <joint name="base_link_joint" type="fixed">

Commit message: fix: base-chassis joint

File: src/catkin_ws/src/jackal-custom/urdf/custom_jackal_base.urdf.xacro (robot description, xacro)
@@ -82,5 +82,5 @@
   <link name="base_link"></link>
   <joint name="base_link_joint" type="fixed">
-    <origin xyz="0 0 0" rpy="0 0 0" />
+    <origin xyz="-0.19 0 -0.184" rpy="0 0 0" />
     <parent link="base_link"/>
     <child link="chassis_link" />

File: src/catkin_ws/src/jackal-custom/urdf/custom_jackal_base_real.urdf.xacro (robot description, xacro)
@@ -63,5 +63,5 @@
   <link name="base_link"></link>
   <joint name="base_link_joint" type="fixed">
-    <origin xyz="0 0 0" rpy="0 0 0" />
+    <origin xyz="-0.19 0 -0.184" rpy="0 0 0" />
     <parent link="base_link"/>
     <child link="chassis_link" />
