Commit message: test: fix joints rvoz

File: src/catkin_ws/src/jackal-custom/urdf/custom_jackal_base_real.urdf.xacro (robot description, xacro)
@@ -116,4 +116,9 @@
     </link>
   </xacro:unless>
+  <joint name="front_fender_joint" type="fixed">
+    <origin xyz="0 0 0" rpy="0 0 0"/>
+    <parent link="chassis_link" />
+    <child link="front_fender_link" />
+  </joint>
   <xacro:if value="$(optenv JACKAL_FRONT_ACCESSORY_FENDER 0)">
     <link name="front_fender_link">
@@ -132,9 +137,4 @@
     </joint>
   </xacro:if>
-  <joint name="front_fender_joint" type="fixed">
-    <origin xyz="0 0 0" rpy="0 0 0"/>
-    <parent link="chassis_link" />
-    <child link="front_fender_link" />
-  </joint>
   <xacro:unless value="$(optenv JACKAL_REAR_ACCESSORY_FENDER 0)">
     <link name="rear_fender_link">
@@ -147,4 +147,9 @@
     </link>
   </xacro:unless>
+  <joint name="rear_fender_joint" type="fixed">
+    <origin xyz="0 0 0" rpy="0 0 ${PI}"/>
+    <parent link="chassis_link" />
+    <child link="rear_fender_link" />
+  </joint>
   <xacro:if value="$(optenv JACKAL_REAR_ACCESSORY_FENDER 0)">
     <link name="rear_fender_link">
@@ -163,9 +168,4 @@
     </joint>
   </xacro:if>
-  <joint name="rear_fender_joint" type="fixed">
-    <origin xyz="0 0 0" rpy="0 0 ${PI}"/>
-    <parent link="chassis_link" />
-    <child link="rear_fender_link" />
-  </joint>
   <!-- IMU LINK -->
   <link name="imu_link">

Commit message: test: fix views rviz

File: src/catkin_ws/src/jackal-custom/urdf/custom_jackal_base_real.urdf.xacro (robot description, xacro)
@@ -41,18 +41,18 @@
       </inertial>
     </link>
-    <joint name="${prefix}_wheel" type="continuous">
+    <joint name="${prefix}_wheel" type="fixed">
       <parent link="chassis_link"/>
       <child link="${prefix}_wheel_link" />
       <xacro:insert_block name="joint_pose" />
-      <axis xyz="0 1 0" />
     </joint>
   </xacro:macro>
   <!---->
   <link name="world"></link>
-  <joint name="world_joint" type="fixed">
+  <joint name="world_joint" type="continuous">
     <origin xyz="0 0 0" rpy="0 0 0" />
     <parent link="world"/>
     <child link="odom" />
     <update_rate value="50" />
+    <axis xyz="0 1 0" />
   </joint>
   <link name="odom"></link>

Commit message: chore: test orientation

File: src/catkin_ws/src/jackal-custom/urdf/custom_jackal_base_real.urdf.xacro (robot description, xacro)
@@ -41,16 +41,16 @@
       </inertial>
     </link>
-    <joint name="${prefix}_wheel" type="continuous">
+    <joint name="${prefix}_wheel" type="fixed">
       <parent link="chassis_link"/>
       <child link="${prefix}_wheel_link" />
       <xacro:insert_block name="joint_pose" />
-      <axis xyz="0 1 0" />
     </joint>
   </xacro:macro>
   <link name="world"></link>
-  <joint name="world_joint" type="fixed">
+  <joint name="world_joint" type="continuous">
     <origin xyz="0 0 0" rpy="0 0 0" />
     <parent link="world"/>
     <child link="world" />
+    <axis xyz="0 1 0" />
   </joint>
   <link name="odom"></link>

Commit message: chore: uwb colors

File: src/catkin_ws/src/jackal-custom/urdf/custom_jackal_base_real.urdf.xacro (robot description, xacro)
@@ -215,5 +215,5 @@
        of these into the final description is controlled by optenv variables, which
        default each one to off.-->
-  <xacro:include filename="$(find jackal_description)/urdf/accessories.urdf.xacro" />
+  <!--xacro:include filename="$(find jackal_description)/urdf/accessories.urdf.xacro" /-->
   <!-- Optional custom includes. -->
   <xacro:include filename="$(optenv JACKAL_URDF_EXTRAS empty.urdf)" />

File: src/catkin_ws/src/jackal-custom/urdf/custom_jackal_real.urdf.xacro (robot description, xacro)
@@ -26,7 +26,7 @@
                 <mesh filename="package://jackal-custom/models/DecaWave/meshes/Decawave.stl"/>
             </geometry>
-            <material name="right_tag_color">
+            <!--material name="right_tag_color">
                 <color rgba="200 0 0 0"/>
-            </material>
+            </material-->
         </visual>
     </link>
@@ -44,5 +44,5 @@
         </inertial>
         <collision>
-            <origin xyz="0 -0.013 0" rpy="-1.57 0 1.57"/>
+            <origin xyz="0 -0.013 0" rpy="0 0 0"/>
             <geometry>
                 <box size="0.05 0.026 0.102"/>
@@ -50,11 +50,11 @@
         </collision>
         <visual>
-            <origin xyz="0 0 0" rpy="0 0 3.14159265359"/>
+            <origin xyz="0 0 0" rpy="-1.57 0 -1.57"/>
             <geometry>
                 <mesh filename="package://jackal-custom/models/DecaWave/meshes/Decawave.stl"/>
             </geometry>
-            <material name="left_tag_color">
+            <!--material name="left_tag_color">
                 <color rgba="0 200 0 0"/>
-            </material>
+            </material-->
         </visual>
     </link>
@@ -82,7 +82,7 @@
                 <mesh filename="package://jackal-custom/models/DecaWave/meshes/Decawave.stl"/>
             </geometry>
-            <material name="rear_tag_color">
+            <!--material name="rear_tag_color">
                 <color rgba="0 0 200 0"/>
-            </material>
+            </material-->
         </visual>
     </link>

Commit message: fix: real urdf

File: src/catkin_ws/src/jackal-custom/urdf/custom_jackal_base_real.urdf.xacro (robot description, xacro)
@@ -63,5 +63,5 @@
   <link name="base_link"></link>
   <joint name="base_link_joint" type="fixed">
-    <origin xyz="-0.19 0 -0.184" rpy="0 0 0" />
+    <origin xyz="0 0 0" rpy="0 0 0" />
     <parent link="base_link"/>
     <child link="chassis_link" />

File: src/catkin_ws/src/jackal-custom/urdf/custom_jackal_real.urdf.xacro (robot description, xacro)
@@ -39,5 +39,5 @@
     <joint name="right_tag_joint" type="fixed">
         <origin xyz="0.095 0.164 0.184" rpy="0 0 0"/>
-        <parent link="base_link"/>
+        <parent link="chassis_link"/>
         <child link="right_tag"/>
     </joint>
@@ -67,5 +67,5 @@
     <joint name="left_tag_joint" type="fixed">
         <origin xyz="0.095 -0.164 0.184" rpy="0 0 0"/>
-        <parent link="base_link"/>
+        <parent link="chassis_link"/>
         <child link="left_tag"/>
     </joint>
@@ -95,5 +95,5 @@
     <joint name="rear_tag_joint" type="fixed">
         <origin xyz="-0.19 0.0 0.184" rpy="0 0 0"/>
-        <parent link="base_link"/>
+        <parent link="chassis_link"/>
         <child link="rear_tag"/>
     </joint>
