Commit message: feat: working UWB real

File: src/catkin_ws/src/jackal-custom/urdf/custom_jackal_real.urdf.xacro (robot description, xacro)
@@ -81,5 +81,5 @@
     </link>
     <joint name="rear_tag_joint" type="fixed">
-        <origin xyz="-0.5 0 0.184" rpy="0 0 0"/>
+        <origin xyz="-0.15 0 0.184" rpy="0 0 0"/>
         <!--origin xyz="0 0 0.184" rpy="0 0 0"/-->
         <parent link="base_link"/>

Commit message: test: fixed tag

File: src/catkin_ws/src/jackal-custom/urdf/custom_jackal_real.urdf.xacro (robot description, xacro)
@@ -74,5 +74,5 @@
         </collision>
         <visual>
-            <origin xyz="0 0 0" rpy="0 0 -1.57"/>
+            <origin xyz="0 0 0" rpy="1.57 0 -1.57"/>
             <geometry>
                 <mesh filename="package://jackal-custom/models/DecaWave/meshes/Decawave.stl"/>
@@ -81,5 +81,5 @@
     </link>
     <joint name="rear_tag_joint" type="fixed">
-        <origin xyz="-0.15 0 0.184" rpy="0 0 0"/>
+        <origin xyz="0.12 0.10 0.225" rpy="0 0 0"/>
         <!--origin xyz="0 0 0.184" rpy="0 0 0"/-->
         <parent link="base_link"/>

Commit message: test: fixed tag

File: src/catkin_ws/src/jackal-custom/urdf/custom_jackal_real.urdf.xacro (robot description, xacro)
@@ -74,5 +74,5 @@
         </collision>
         <visual>
-            <origin xyz="0 0 0" rpy="1.57 0 -1.57"/>
+            <origin xyz="0 0 0" rpy="-1.57 0 -1.57"/>
             <geometry>
                 <mesh filename="package://jackal-custom/models/DecaWave/meshes/Decawave.stl"/>
@@ -81,5 +81,5 @@
     </link>
     <joint name="rear_tag_joint" type="fixed">
-        <origin xyz="0.12 0.10 0.225" rpy="0 0 0"/>
+        <origin xyz="-0.12 -0.10 0.225" rpy="0 0 0"/>
         <!--origin xyz="0 0 0.184" rpy="0 0 0"/-->
         <parent link="base_link"/>

Commit message: test: fixed tag

File: src/catkin_ws/src/jackal-custom/urdf/custom_jackal_real.urdf.xacro (robot description, xacro)
@@ -81,5 +81,5 @@
     </link>
     <joint name="rear_tag_joint" type="fixed">
-        <origin xyz="-0.12 -0.10 0.225" rpy="0 0 0"/>
+        <origin xyz="0.12 0.10 0.225" rpy="0 0 0"/>
         <!--origin xyz="0 0 0.184" rpy="0 0 0"/-->
         <parent link="base_link"/>

Commit message: chore: urdf change

File: src/catkin_ws/src/jackal-custom/urdf/custom_jackal_real.urdf.xacro (robot description, xacro)
@@ -29,5 +29,5 @@
     </link>
     <joint name="right_tag_joint" type="fixed">
-        <origin xyz="0.05 -0.14 0.28" rpy="0 0 0"/>
+        <origin xyz="0.19 -0.35 0.184" rpy="0 0 0"/>
         <parent link="base_link"/>
         <child link="right_tag"/>
@@ -54,5 +54,5 @@
     </link>
     <joint name="left_tag_joint" type="fixed">
-        <origin xyz="0.05 0.14 0.28" rpy="0 0 0"/>
+        <origin xyz="0.19 0.35 0.184" rpy="0 0 0"/>
         <parent link="base_link"/>
         <child link="left_tag"/>
@@ -79,5 +79,5 @@
     </link>
     <joint name="rear_tag_joint" type="fixed">
-        <origin xyz="-0.14 0.0 0.28" rpy="0 0 0"/>
+        <origin xyz="-0.45 0.0 0.184" rpy="0 0 0"/>
         <parent link="base_link"/>
         <child link="rear_tag"/>

Commit message: chore: uwb colors

File: src/catkin_ws/src/jackal-custom/urdf/custom_jackal_real.urdf.xacro (robot description, xacro)
@@ -22,8 +22,11 @@
         </collision>
         <visual>
-            <origin xyz="0 0 0" rpy="0 0 0"/>
+            <origin xyz="0 0 0" rpy="-1.57 0 -1.57"/>
             <geometry>
                 <mesh filename="package://jackal-custom/models/DecaWave/meshes/Decawave.stl"/>
             </geometry>
+            <material>
+                <color rgba="200 0 0 0"/>
+            </material>
         </visual>
     </link>
@@ -41,5 +44,5 @@
         </inertial>
         <collision>
-            <origin xyz="0 -0.013 0" rpy="0 0 0"/>
+            <origin xyz="0 -0.013 0" rpy="-1.57 0 1.57"/>
             <geometry>
                 <box size="0.05 0.026 0.102"/>
@@ -51,4 +54,7 @@
                 <mesh filename="package://jackal-custom/models/DecaWave/meshes/Decawave.stl"/>
             </geometry>
+            <material>
+                <color rgba="0 200 0 0"/>
+            </material>
         </visual>
     </link>
@@ -76,8 +82,11 @@
                 <mesh filename="package://jackal-custom/models/DecaWave/meshes/Decawave.stl"/>
             </geometry>
+            <material>
+                <color rgba="0 0 200 0"/>
+            </material>
         </visual>
     </link>
     <joint name="rear_tag_joint" type="fixed">
-        <origin xyz="-0.45 0.0 0.184" rpy="0 0 0"/>
+        <origin xyz="-0.18 0.0 0.184" rpy="0 0 0"/>
         <parent link="base_link"/>
         <child link="rear_tag"/>

Commit message: chore: uwb colors

File: src/catkin_ws/src/jackal-custom/urdf/custom_jackal_real.urdf.xacro (robot description, xacro)
@@ -26,5 +26,5 @@
                 <mesh filename="package://jackal-custom/models/DecaWave/meshes/Decawave.stl"/>
             </geometry>
-            <material>
+            <material name="right_tag_color">
                 <color rgba="200 0 0 0"/>
             </material>
@@ -54,5 +54,5 @@
                 <mesh filename="package://jackal-custom/models/DecaWave/meshes/Decawave.stl"/>
             </geometry>
-            <material>
+            <material name="left_tag_color">
                 <color rgba="0 200 0 0"/>
             </material>
@@ -82,5 +82,5 @@
                 <mesh filename="package://jackal-custom/models/DecaWave/meshes/Decawave.stl"/>
             </geometry>
-            <material>
+            <material name="rear_tag_color">
                 <color rgba="0 0 200 0"/>
             </material>

Commit message: feat: vicon position and orientation

File: src/catkin_ws/src/jackal-custom/urdf/custom_jackal_real.urdf.xacro (robot description, xacro)
@@ -8,4 +8,10 @@
     <xacro:property name="right" value="$(arg right_id)" />
     <xacro:property name="left" value="$(arg left_id)" />
+    <link name="vicon_link"></link>
+    <joint name="vicon_link_joint" type="fixed">
+      <origin xyz="0 0 0.184" rpy="0 0 0" />
+      <parent link="base_link"/>
+      <child link="vicon_link" />
+    </joint>
     <!-- -->
     <link name="right_tag">

Commit message: test: wider tags for orientation

File: src/catkin_ws/src/jackal-custom/urdf/custom_jackal_real.urdf.xacro (robot description, xacro)
@@ -38,5 +38,5 @@
     </link>
     <joint name="right_tag_joint" type="fixed">
-        <origin xyz="0.095 0.164 0.184" rpy="0 0 0"/>
+        <origin xyz="0.15 0.25 0.184" rpy="0 0 0"/>
         <parent link="chassis_link"/>
         <child link="right_tag"/>
@@ -66,5 +66,5 @@
     </link>
     <joint name="left_tag_joint" type="fixed">
-        <origin xyz="0.095 -0.164 0.184" rpy="0 0 0"/>
+        <origin xyz="0.15 -0.25 0.184" rpy="0 0 0"/>
         <parent link="chassis_link"/>
         <child link="left_tag"/>
@@ -94,5 +94,5 @@
     </link>
     <joint name="rear_tag_joint" type="fixed">
-        <origin xyz="-0.19 0.0 0.184" rpy="0 0 0"/>
+        <origin xyz="-0.30 0.0 0.184" rpy="0 0 0"/>
         <parent link="chassis_link"/>
         <child link="rear_tag"/>

Commit message: chore: urdf tags

File: src/catkin_ws/src/jackal-custom/urdf/custom_jackal_real.urdf.xacro (robot description, xacro)
@@ -38,5 +38,5 @@
     </link>
     <joint name="right_tag_joint" type="fixed">
-        <origin xyz="0.15 0.25 0.184" rpy="0 0 0"/>
+        <origin xyz="0.15 -0.25 0.184" rpy="0 0 0"/>
         <parent link="chassis_link"/>
         <child link="right_tag"/>
@@ -66,5 +66,5 @@
     </link>
     <joint name="left_tag_joint" type="fixed">
-        <origin xyz="0.15 -0.25 0.184" rpy="0 0 0"/>
+        <origin xyz="0.15 0.25 0.184" rpy="0 0 0"/>
         <parent link="chassis_link"/>
         <child link="left_tag"/>

Commit message: chore: urdf vicon joint

File: src/catkin_ws/src/jackal-custom/urdf/custom_jackal_real.urdf.xacro (robot description, xacro)
@@ -10,5 +10,5 @@
     <link name="vicon_link"></link>
     <joint name="vicon_link_joint" type="fixed">
-      <origin xyz="0 0 0.184" rpy="0 0 0" />
+      <origin xyz="0.085 0 0.184" rpy="0 0 0" />
       <parent link="base_link"/>
       <child link="vicon_link" />
